Commit message: working with gazebo on simulation only, ros  working with physical robot, working on moveit integration

File: melfa_description/urdf/rv4fl.urdf.xacro (robot description, xacro)
@@ -10,3 +10,7 @@
     <origin xyz="0 0 0" rpy="0 0 0"/>
   </xacro:rv4fl>
+  <xacro:include filename="rv4fl_gazebo.xacro"/>
+  <xacro:rv4fl_gazebo arm_id="first"/>
+  <xacro:include filename="rv4fl_control.xacro"/>
+  <xacro:rv4fl_control arm_id="first"/>
 </robot>

File: melfa_description/urdf/rv4fl.xacro (robot description, xacro)
@@ -2,4 +2,5 @@
 <!-- Copyright (C) 2018, Tokyo Opensource Robotics Kyokai Association -->
 <robot xmlns:xacro="http://www.ros.org/wiki/xacro">
+  <xacro:property name="inertial" value="${xacro.load_yaml('rv4fl_inertial.yaml')}" />
   <xacro:macro name="rv4fl" params="parent *origin">
     <joint name="rv4fl_mounting_joint" type="fixed">
@@ -10,16 +11,23 @@
     <link name="link0">
       <visual>
-	<origin rpy="0 0 ${pi}" xyz="0 0 0"/>
-	<geometry>
-	  <mesh filename="package://melfa_description/mesh/rv4fl/L0.stl"/>
-	</geometry>
-	<material name="white"/>
-      </visual>
-      <collision>
-	<origin rpy="0 0 ${pi}" xyz="0 0 0"/>
-	<geometry>
-	  <mesh filename="package://melfa_description/mesh/rv4fl/L0.stl"/>
-	</geometry>
-      </collision>
+        <origin rpy="0 0 ${pi}" xyz="0 0 0"/>
+        <geometry>
+          <mesh filename="package://melfa_description/mesh/rv4fl/L0.stl"/>
+        </geometry>
+        <material name="white"/>
+      </visual>
+      <collision>
+        <origin rpy="0 0 ${pi}" xyz="0 0 0"/>
+        <geometry>
+          <mesh filename="package://melfa_description/mesh/rv4fl/L0.stl"/>
+        </geometry>
+      </collision>
+      <inertial>
+        <origin rpy="0 0 0" xyz="0 0 0"/>
+        <mass value="${inertial['link_0_mass']}"/>
+        <inertia ixx="${inertial['link_0_inertia']['ixx']}" ixy="${inertial['link_0_inertia']['ixy']}" ixz="${inertial['link_0_inertia']['ixz']}"
+            iyy="${inertial['link_0_inertia']['iyy']}" iyz="${inertial['link_0_inertia']['iyz']}"
+            izz="${inertial['link_0_inertia']['izz']}"/>
+      </inertial>
     </link>
     <joint name="joint1" type="revolute">
@@ -33,16 +41,23 @@
     <link name="link1">
       <visual>
-	<origin rpy="0 0 0" xyz="0 0 -0.350"/>
-	<geometry>
-	  <mesh filename="package://melfa_description/mesh/rv4fl/L1.stl"/>
-	</geometry>
-	<material name="white"/>
-      </visual>
-      <collision>
-	<origin rpy="0 0 0" xyz="0 0 -0.350"/>
-	<geometry>
-	  <mesh filename="package://melfa_description/mesh/rv4fl/L1.stl"/>
-	</geometry>
-      </collision>
+        <origin rpy="0 0 0" xyz="0 0 -0.350"/>
+        <geometry>
+          <mesh filename="package://melfa_description/mesh/rv4fl/L1.stl"/>
+        </geometry>
+        <material name="white"/>
+      </visual>
+      <collision>
+        <origin rpy="0 0 0" xyz="0 0 -0.350"/>
+        <geometry>
+          <mesh filename="package://melfa_description/mesh/rv4fl/L1.stl"/>
+        </geometry>
+      </collision>
+      <inertial>
+        <origin rpy="0 0 0" xyz="0 0 0"/>
+        <mass value="${inertial['link_1_mass']}"/>
+        <inertia ixx="${inertial['link_1_inertia']['ixx']}" ixy="${inertial['link_1_inertia']['ixy']}" ixz="${inertial['link_1_inertia']['ixz']}"
+            iyy="${inertial['link_1_inertia']['iyy']}" iyz="${inertial['link_1_inertia']['iyz']}"
+            izz="${inertial['link_1_inertia']['izz']}"/>
+      </inertial>
     </link>
     <joint name="joint2" type="revolute">
@@ -56,16 +71,23 @@
     <link name="link2">
       <visual>
-	<origin rpy="0 0 ${pi}" xyz="0 0 -0.350"/>
-	<geometry>
-	  <mesh filename="package://melfa_description/mesh/rv4fl/L2.stl"/>
-	</geometry>
-	<material name="white"/>
-      </visual>
-      <collision>
-	<origin rpy="0 0 ${pi}" xyz="0 0 -0.350"/>
-	<geometry>
-	  <mesh filename="package://melfa_description/mesh/rv4fl/L2.stl"/>
-	</geometry>
-      </collision>
+        <origin rpy="0 0 ${pi}" xyz="0 0 -0.350"/>
+        <geometry>
+          <mesh filename="package://melfa_description/mesh/rv4fl/L2.stl"/>
+        </geometry>
+        <material name="white"/>
+      </visual>
+      <collision>
+        <origin rpy="0 0 ${pi}" xyz="0 0 -0.350"/>
+        <geometry>
+          <mesh filename="package://melfa_description/mesh/rv4fl/L2.stl"/>
+        </geometry>
+      </collision>
+      <inertial>
+        <origin rpy="0 0 0" xyz="0 0 0"/>
+        <mass value="${inertial['link_2_mass']}"/>
+        <inertia ixx="${inertial['link_2_inertia']['ixx']}" ixy="${inertial['link_2_inertia']['ixy']}" ixz="${inertial['link_2_inertia']['ixz']}"
+            iyy="${inertial['link_2_inertia']['iyy']}" iyz="${inertial['link_2_inertia']['iyz']}"
+            izz="${inertial['link_2_inertia']['izz']}"/>
+      </inertial>
     </link>
     <joint name="joint3" type="revolute">
@@ -79,16 +101,23 @@
     <link name="link3">
       <visual>
-	<origin rpy="0 0 ${pi}" xyz="0 0 ${-0.350-0.310}"/>
-	<geometry>
-	  <mesh filename="package://melfa_description/mesh/rv4fl/L3.stl"/>
-	</geometry>
-	<material name="white"/>
-      </visual>
-      <collision>
-	<origin rpy="0 0 ${pi}" xyz="0 0 ${-0.350-0.310}"/>
-	<geometry>
-	  <mesh filename="package://melfa_description/mesh/rv4fl/L3.stl"/>
-	</geometry>
-      </collision>
+        <origin rpy="0 0 ${pi}" xyz="0 0 ${-0.350-0.310}"/>
+        <geometry>
+          <mesh filename="package://melfa_description/mesh/rv4fl/L3.stl"/>
+        </geometry>
+        <material name="white"/>
+      </visual>
+      <collision>
+        <origin rpy="0 0 ${pi}" xyz="0 0 ${-0.350-0.310}"/>
+        <geometry>
+          <mesh filename="package://melfa_description/mesh/rv4fl/L3.stl"/>
+        </geometry>
+      </collision>
+      <inertial>
+        <origin rpy="0 0 0" xyz="0 0 0"/>
+        <mass value="${inertial['link_3_mass']}"/>
+        <inertia ixx="${inertial['link_3_inertia']['ixx']}" ixy="${inertial['link_3_inertia']['ixy']}" ixz="${inertial['link_3_inertia']['ixz']}"
+            iyy="${inertial['link_3_inertia']['iyy']}" iyz="${inertial['link_3_inertia']['iyz']}"
+            izz="${inertial['link_3_inertia']['izz']}"/>
+      </inertial>
     </link>
     <joint name="joint4" type="revolute">
@@ -102,16 +131,23 @@
     <link name="link4">
       <visual>
-	<origin rpy="0 0 0" xyz="-0.050 0 ${-0.350-0.310-0.335}"/>
-	<geometry>
-	  <mesh filename="package://melfa_description/mesh/rv4fl/L4.stl"/>
-	</geometry>
-	<material name="white"/>
-      </visual>
-      <collision>
-	<origin rpy="0 0 0" xyz="-0.050 0 ${-0.350-0.310-0.335}"/>
-	<geometry>
-	  <mesh filename="package://melfa_description/mesh/rv4fl/L4.stl"/>
-	</geometry>
-      </collision>
+        <origin rpy="0 0 0" xyz="-0.050 0 ${-0.350-0.310-0.335}"/>
+        <geometry>
+          <mesh filename="package://melfa_description/mesh/rv4fl/L4.stl"/>
+        </geometry>
+        <material name="white"/>
+      </visual>
+      <collision>
+        <origin rpy="0 0 0" xyz="-0.050 0 ${-0.350-0.310-0.335}"/>
+        <geometry>
+          <mesh filename="package://melfa_description/mesh/rv4fl/L4.stl"/>
+        </geometry>
+      </collision>
+      <inertial>
+        <origin rpy="0 0 0" xyz="0 0 0"/>
+        <mass value="${inertial['link_4_mass']}"/>
+        <inertia ixx="${inertial['link_4_inertia']['ixx']}" ixy="${inertial['link_4_inertia']['ixy']}" ixz="${inertial['link_4_inertia']['ixz']}"
+            iyy="${inertial['link_4_inertia']['iyy']}" iyz="${inertial['link_4_inertia']['iyz']}"
+            izz="${inertial['link_4_inertia']['izz']}"/>
+      </inertial>
     </link>
     <joint name="joint5" type="revolute">
@@ -125,16 +161,23 @@
     <link name="link5">
       <visual>
-	<origin rpy="0 0 0" xyz="-0.050 0 ${-0.350-0.310-0.335}"/>
-	<geometry>
-	  <mesh filename="package://melfa_description/mesh/rv4fl/L5.stl"/>
-	</geometry>
-	<material name="white"/>
-      </visual>
-      <collision>
-	<origin rpy="0 0 0" xyz="-0.050 0 ${-0.350-0.310-0.335}"/>
-	<geometry>
-	  <mesh filename="package://melfa_description/mesh/rv4fl/L5.stl"/>
-	</geometry>
-      </collision>
+        <origin rpy="0 0 0" xyz="-0.050 0 ${-0.350-0.310-0.335}"/>
+        <geometry>
+          <mesh filename="package://melfa_description/mesh/rv4fl/L5.stl"/>
+        </geometry>
+        <material name="white"/>
+      </visual>
+      <collision>
+        <origin rpy="0 0 0" xyz="-0.050 0 ${-0.350-0.310-0.335}"/>
+        <geometry>
+          <mesh filename="package://melfa_description/mesh/rv4fl/L5.stl"/>
+        </geometry>
+      </collision>
+      <inertial>
+        <origin rpy="0 0 0" xyz="0 0 0"/>
+        <mass value="${inertial['link_5_mass']}"/>
+        <inertia ixx="${inertial['link_5_inertia']['ixx']}" ixy="${inertial['link_5_inertia']['ixy']}" ixz="${inertial['link_5_inertia']['ixz']}"
+            iyy="${inertial['link_5_inertia']['iyy']}" iyz="${inertial['link_5_inertia']['iyz']}"
+            izz="${inertial['link_5_inertia']['izz']}"/>
+      </inertial>
     </link>
     <joint name="joint6" type="revolute">
@@ -148,16 +191,23 @@
     <link name="link6">
       <visual>
-	<origin rpy="0 0 0" xyz="-0.050 0 ${-0.350-0.310-0.335-0.125}"/>
-	<geometry>
-	  <mesh filename="package://melfa_description/mesh/rv4fl/L6.stl"/>
-	</geometry>
-	<material name="white"/>
-      </visual>
-      <collision>
-	<origin rpy="0 0 0" xyz="-0.050 0 ${-0.350-0.310-0.335-0.125}"/>
-	<geometry>
-	  <mesh filename="package://melfa_description/mesh/rv4fl/L6.stl"/>
-	</geometry>
-      </collision>
+        <origin rpy="0 0 0" xyz="-0.050 0 ${-0.350-0.310-0.335-0.125}"/>
+        <geometry>
+          <mesh filename="package://melfa_description/mesh/rv4fl/L6.stl"/>
+        </geometry>
+        <material name="white"/>
+      </visual>
+      <collision>
+        <origin rpy="0 0 0" xyz="-0.050 0 ${-0.350-0.310-0.335-0.125}"/>
+        <geometry>
+          <mesh filename="package://melfa_description/mesh/rv4fl/L6.stl"/>
+        </geometry>
+      </collision>
+      <inertial>
+        <origin rpy="0 0 0" xyz="0 0 0"/>
+        <mass value="${inertial['link_6_mass']}"/>
+        <inertia ixx="${inertial['link_6_inertia']['ixx']}" ixy="${inertial['link_6_inertia']['ixy']}" ixz="${inertial['link_6_inertia']['ixz']}"
+            iyy="${inertial['link_6_inertia']['iyy']}" iyz="${inertial['link_6_inertia']['iyz']}"
+            izz="${inertial['link_6_inertia']['izz']}"/>
+      </inertial>
     </link>
   </xacro:macro>
