Commit message: tweaking physical properties of the robot model

File: melfa_description/urdf/rv4fl.xacro (robot description, xacro)
@@ -24,5 +24,5 @@
       </collision>
       <inertial>
-        <origin rpy="0 0 0" xyz="0 0 0"/>
+        <origin rpy="0 0 ${pi}" xyz= "0.028955 -0.001000 0.095391"/>
         <mass value="${inertial['link_0_mass']}"/>
         <inertia ixx="${inertial['link_0_inertia']['ixx']}" ixy="${inertial['link_0_inertia']['ixy']}" ixz="${inertial['link_0_inertia']['ixz']}"
@@ -54,5 +54,5 @@
       </collision>
       <inertial>
-        <origin rpy="0 0 0" xyz="0 0 0"/>
+        <origin rpy="0 0 0" xyz="0.003199 0.000002 ${-0.35+0.28392}"/>
         <mass value="${inertial['link_1_mass']}"/>
         <inertia ixx="${inertial['link_1_inertia']['ixx']}" ixy="${inertial['link_1_inertia']['ixy']}" ixz="${inertial['link_1_inertia']['ixz']}"
@@ -84,5 +84,5 @@
       </collision>
       <inertial>
-        <origin rpy="0 0 0" xyz="0 0 0"/>
+        <origin rpy="0 0 0" xyz="0.017161 0.0 ${-0.35+0.460138}"/>
         <mass value="${inertial['link_2_mass']}"/>
         <inertia ixx="${inertial['link_2_inertia']['ixx']}" ixy="${inertial['link_2_inertia']['ixy']}" ixz="${inertial['link_2_inertia']['ixz']}"
@@ -114,5 +114,5 @@
       </collision>
       <inertial>
-        <origin rpy="0 0 0" xyz="0 0 0"/>
+        <origin rpy="0 0 0" xyz="0.024203 0.000348  ${-0.350-0.310+0.652442}"/>
         <mass value="${inertial['link_3_mass']}"/>
         <inertia ixx="${inertial['link_3_inertia']['ixx']}" ixy="${inertial['link_3_inertia']['ixy']}" ixz="${inertial['link_3_inertia']['ixz']}"
@@ -144,5 +144,5 @@
       </collision>
       <inertial>
-        <origin rpy="0 0 0" xyz="0 0 0"/>
+        <origin rpy="0 0 0" xyz="${-0.050+0.050518} -0.000053 ${-0.350-0.310-0.335+0.856493}"/>
         <mass value="${inertial['link_4_mass']}"/>
         <inertia ixx="${inertial['link_4_inertia']['ixx']}" ixy="${inertial['link_4_inertia']['ixy']}" ixz="${inertial['link_4_inertia']['ixz']}"
@@ -174,5 +174,5 @@
       </collision>
       <inertial>
-        <origin rpy="0 0 0" xyz="0 0 0"/>
+        <origin rpy="0 0 0" xyz="${-0.050+0.050000} 0.0 ${-0.350-0.310-0.335+1.015771}"/>
         <mass value="${inertial['link_5_mass']}"/>
         <inertia ixx="${inertial['link_5_inertia']['ixx']}" ixy="${inertial['link_5_inertia']['ixy']}" ixz="${inertial['link_5_inertia']['ixz']}"
@@ -204,5 +204,5 @@
       </collision>
       <inertial>
-        <origin rpy="0 0 0" xyz="0 0 0"/>
+        <origin rpy="0 0 0" xyz="${-0.050+0.050000} 0.0 ${-0.350-0.310-0.335-0.125+1.105770}"/>
         <mass value="${inertial['link_6_mass']}"/>
         <inertia ixx="${inertial['link_6_inertia']['ixx']}" ixy="${inertial['link_6_inertia']['ixy']}" ixz="${inertial['link_6_inertia']['ixz']}"
